File: kicad/TL082CP/power.kicad_sch (KiCad schematic)
At the start: 1 part, among them U1 TMR_1-1222

Commit message: fix: schematic capacitors, resistors, symbols updated
Parts:
- added C5, C6: 100nF, Capacitor_THT:C_Disc_D5.0mm_W2.5mm_P5.00mm, symbol Device:C
Connections:
- net +12V: now also C5.1
- net -12V: now also C6.1
- net GND: now also C5.2, C6.2
