File: kicad/TL082CP/TL082CP.kicad_sch (KiCad schematic)
At the start: 3 parts, among them J1 AudioJack2_Switch, J2 AudioJack2_Switch, J4 Barrel_Jack

Commit message: fix: schematic capacitors, resistors, symbols updated
Parts:
- removed J4: Barrel_Jack, Connector_BarrelJack:BarrelJack_SwitchcraftConxall_RAPC10U_Horizontal, symbol Connector:Barrel_Jack
- added J3: PJ-102A, PJ-102A:CUI_PJ-102A, symbol 1_own_PJ-102A:PJ-102A
Connections:
- net dual supply voltage/+VIN: now also J3.1
- net dual supply voltage/-VIN: now also J3.2
- no-connect marks 4 -> 5
Other:
- note added: "Audio Preamp Main"
- note removed: "Guitar Preamp Main"

Commit message: final pcb layout and updated doc
Parts:
- J3: footprint PJ-102A:CUI_PJ-102A -> 1_own_PJ-102A:CUI_PJ-102A
Changed lines of the file:
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@@
 			)
 		)
-		(property "Footprint" "PJ-102A:CUI_PJ-102A"
+		(property "Footprint" "1_own_PJ-102A:CUI_PJ-102A"
 			(at 102.87 41.91 0)
 			(effects
